File: Hardware/MSPBMP/MSPBMP.sch (KiCad schematic (older format))
At the start: 49 parts, among them J1 USB_B_Micro, J2 SWD, J3 RS232, J4 JTAG, J5 ISP, U1 MCP1700T-3302E/TT, U2 STM32F103CBT6, U3 LM358DR2G, U4 TXS0108EPWR, Y1 8MHz

Commit message: Schematics and PCB review
Parts:
- added C22: 100nF, Capacitor_SMD:C_0603_1608Metric_Pad1.08x0.95mm_HandSolder, symbol Device:C
- added R15: 47K, Resistor_SMD:R_0603_1608Metric_Pad0.98x0.95mm_HandSolder, symbol Device:R
- R5: Descr Chip Resistor - Surface Mount 10KOhms ±1% 1/10W 0603 RoHS -> 100Ω ±1% 1/10W ±200ppm/°C 0603 Chip Resistor - Surface Moun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; LCSC C25804 -> C22775
- U1: value MCP1700T-3302E/TT -> AMS1117-3.3; footprint Package_TO_SOT_SMD:SOT-23 -> Package_TO_SOT_SMD:SOT-223-3_TabPin2; symbol Regulator_Linear:MCP1700-3302E_SOT23 -> Regulator_Linear:AMS1117-3.3; Descr MCP1700T-3302E/TT - Fixed 6V 3.3V 350mV @ 250mA SOT-23(SOT-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 -> Fixed 15V 3.3V 1.3V @ 800mA SOT-223 Dropout Regulators(LDO)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; LCSC C39051 -> C6186
Connections:
- wire segments 247 -> 253
Other:
- moved on the sheet: C20, D1, D2, R11, R12, R13, R7, R8

Commit message: More Hardware improvements
Parts:
- added RN1, RN2, RN3: 33, Resistor_SMD:R_Array_Convex_4x0402, symbol Device:R_Pack04
- C12: renamed from C10; value 4.7uF -> 22uF; Descr 4.7uF ±10% 16V X5R 0603 Multilayer Ceramic Capacitors MLCC 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 -> 22uF ±20% 6.3V X5R 0603 Multilayer Ceramic Capacitors MLCC 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; LCSC C19666 -> C59461
- C16: renamed from C14; value 4.7uF -> 22uF; Descr 4.7uF ±10% 16V X5R 0603 Multilayer Ceramic Capacitors MLCC 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 -> 22uF ±20% 6.3V X5R 0603 Multilayer Ceramic Capacitors MLCC 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; LCSC C19666 -> C59461
- C19: renamed from C18; value 4.7uF -> 22uF; Descr 4.7uF ±10% 16V X5R 0603 Multilayer Ceramic Capacitors MLCC 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 -> 22uF ±20% 6.3V X5R 0603 Multilayer Ceramic Capacitors MLCC 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; LCSC C19666 -> C59461
- C2: value 4.7uF -> 10uF; Descr 4.7uF ±10% 16V X5R 0603 Multilayer Ceramic Capacitors MLCC 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 -> 10uF ±10% 10V X5R 0603 Multilayer Ceramic Capacitors MLCC -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; LCSC C19666 -> C19702
- C20: renamed from C19; value 4.7uF -> 22uF; Descr 4.7uF ±10% 16V X5R 0603 Multilayer Ceramic Capacitors MLCC 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 -> 22uF ±20% 6.3V X5R 0603 Multilayer Ceramic Capacitors MLCC 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; LCSC C19666 -> C59461
- C4: value 4.7uF -> 22uF; Descr 4.7uF ±10% 16V X5R 0603 Multilayer Ceramic Capacitors MLCC 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 -> 22uF ±20% 6.3V X5R 0603 Multilayer Ceramic Capacitors MLCC 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; LCSC C19666 -> C59461
- C6: value 100nF -> 470nF; Descr 100nF ±10% 50V X7R 0603 Multilayer Ceramic Capacitors MLCC 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 -> 470nF ±10% 25V X7R 0603 Multilayer Ceramic Capacitors MLCC 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; LCSC C14663 -> C1623
- J1: footprint Connector_USB:USB_Mini-B_Lumberg_2486_01_Horizontal -> lib:USB_Mini-B_Lumberg_2486_01_Horizontal_hand_soldered
- NT1: renamed from R6; footprint Resistor_SMD:R_0603_1608Metric_Pad0.98x0.95mm_HandSolder -> NetTie:NetTie-2_SMD_Pad0.5mm; symbol Device:R -> Device:Net-Tie_2; Descr 0Ω ±1% 0.1W 0603 Chip Resistor - Surface Mount RoHS -> (none); LCSC C21189 -> (none)
- renumbered C9 to C10, C12 to C11, C22 to C14, C16 to C17, C17 to C18, C20 to C22, C11 to C9, R13 to R10, R14 to R11, R11 to R12, R8 to R13, R12 to R14, R7 to R5, R15 to R6, R5 to R7, R9 to R8, R10 to R9, U4 to U3, U3 to U4
Connections:
- net labels added: BRXD, BTXD
- wire segments 253 -> 276
- no-connect marks 19 -> 23
Other:
- moved on the sheet: C1, C10, C11, C12, C13, C14, C15, C16, C17, C18, C19, C2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

Commit message: Hardware: New stick version using a newer MCU
Parts:
- removed RN1: 33, Resistor_SMD:R_Array_Convex_4x0402, symbol Device:R_Pack04
- added C24, C26: 22uF, Capacitor_SMD:C_0603_1608Metric_Pad1.08x0.95mm_HandSolder, symbol Device:C
- added C25: 100nF, Capacitor_SMD:C_0402_1005Metric_Pad0.74x0.62mm_HandSolder, symbol Device:C
- added C4, C5: 20pF, Capacitor_SMD:C_0402_1005Metric_Pad0.74x0.62mm_HandSolder, symbol Device:C
- added FB1, FB2: 600, Resistor_SMD:R_0805_2012Metric_Pad1.20x1.40mm_HandSolder, symbol Device:Ferrite_Bead_Small
- added R15, R16: 330, Resistor_SMD:R_0402_1005Metric_Pad0.72x0.64mm_HandSolder, symbol Device:R
- C1, C3: footprint Capacitor_SMD:C_0603_1608Metric_Pad1.08x0.95mm_HandSolder -> Capacitor_SMD:C_0402_1005Metric_Pad0.74x0.62mm_HandSolder; Descr 100nF ±10% 50V X7R 0603 Multilayer Ceramic Capacitors MLCC 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 -> 100nF ±10% 16V X7R 0402 Multilayer Ceramic Capacitors MLCC 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; LCSC C14663 -> C1525
- C10: renamed from C8; footprint Capacitor_SMD:C_0603_1608Metric_Pad1.08x0.95mm_HandSolder -> Capacitor_SMD:C_0402_1005Metric_Pad0.74x0.62mm_HandSolder; Descr 100nF ±10% 50V X7R 0603 Multilayer Ceramic Capacitors MLCC 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 -> 100nF ±10% 16V X7R 0402 Multilayer Ceramic Capacitors MLCC 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; LCSC C14663 -> C1525
- C11: renamed from C9; footprint Capacitor_SMD:C_0603_1608Metric_Pad1.08x0.95mm_HandSolder -> Capacitor_SMD:C_0402_1005Metric_Pad0.74x0.62mm_HandSolder; Descr 20pF ±5% 50V C0G 0603 Multilayer Ceramic Capacitors MLCC - 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 -> 20pF ±5% 50V C0G 0402 Multilayer Ceramic Capacitors MLCC - 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; LCSC C1648 -> C1554
- C12: renamed from C10; footprint Capacitor_SMD:C_0603_1608Metric_Pad1.08x0.95mm_HandSolder -> Capacitor_SMD:C_0402_1005Metric_Pad0.74x0.62mm_HandSolder; Descr 100nF ±10% 50V X7R 0603 Multilayer Ceramic Capacitors MLCC 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 -> 100nF ±10% 16V X7R 0402 Multilayer Ceramic Capacitors MLCC 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; LCSC C14663 -> C1525
- C13: renamed from C11; footprint Capacitor_SMD:C_0603_1608Metric_Pad1.08x0.95mm_HandSolder -> Capacitor_SMD:C_0402_1005Metric_Pad0.74x0.62mm_HandSolder; Descr 20pF ±5% 50V C0G 0603 Multilayer Ceramic Capacitors MLCC - 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 -> 20pF ±5% 50V C0G 0402 Multilayer Ceramic Capacitors MLCC - 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; LCSC C1648 -> C1554
- C14: renamed from C12; value 22uF -> 10uF; footprint Capacitor_SMD:C_0603_1608Metric_Pad1.08x0.95mm_HandSolder -> Capacitor_SMD:C_0402_1005Metric_Pad0.74x0.62mm_HandSolder; Descr 22uF ±20% 6.3V X5R 0603 Multilayer Ceramic Capacitors MLCC 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 -> 10uF ±20% 6.3V X5R 0402 Multilayer Ceramic Capacitors MLCC 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; LCSC C59461 -> C15525
- C15: renamed from C13; footprint Capacitor_SMD:C_0603_1608Metric_Pad1.08x0.95mm_HandSolder -> Capacitor_SMD:C_0402_1005Metric_Pad0.74x0.62mm_HandSolder; Descr 100nF ±10% 50V X7R 0603 Multilayer Ceramic Capacitors MLCC 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 -> 100nF ±10% 16V X7R 0402 Multilayer Ceramic Capacitors MLCC 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; LCSC C14663 -> C1525
- C16: renamed from C14; footprint Capacitor_SMD:C_0603_1608Metric_Pad1.08x0.95mm_HandSolder -> Capacitor_SMD:C_0402_1005Metric_Pad0.74x0.62mm_HandSolder; Descr 100nF ±10% 50V X7R 0603 Multilayer Ceramic Capacitors MLCC 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 -> 100nF ±10% 16V X7R 0402 Multilayer Ceramic Capacitors MLCC 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; LCSC C14663 -> C1525
- C17: renamed from C15; footprint Capacitor_SMD:C_0603_1608Metric_Pad1.08x0.95mm_HandSolder -> Capacitor_SMD:C_0402_1005Metric_Pad0.74x0.62mm_HandSolder; Descr 100nF ±10% 50V X7R 0603 Multilayer Ceramic Capacitors MLCC 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 -> 100nF ±10% 16V X7R 0402 Multilayer Ceramic Capacitors MLCC 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; LCSC C14663 -> C1525
- C18: renamed from C16; value 22uF -> 10uF; footprint Capacitor_SMD:C_0603_1608Metric_Pad1.08x0.95mm_HandSolder -> Capacitor_SMD:C_0402_1005Metric_Pad0.74x0.62mm_HandSolder; Descr 22uF ±20% 6.3V X5R 0603 Multilayer Ceramic Capacitors MLCC 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 -> 10uF ±20% 6.3V X5R 0402 Multilayer Ceramic Capacitors MLCC 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; LCSC C59461 -> C15525
- C19: renamed from C17; footprint Capacitor_SMD:C_0603_1608Metric_Pad1.08x0.95mm_HandSolder -> Capacitor_SMD:C_0402_1005Metric_Pad0.74x0.62mm_HandSolder; Descr 100nF ±10% 50V X7R 0603 Multilayer Ceramic Capacitors MLCC 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 -> 100nF ±10% 16V X7R 0402 Multilayer Ceramic Capacitors MLCC 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; LCSC C14663 -> C1525
- C20: renamed from C18; footprint Capacitor_SMD:C_0603_1608Metric_Pad1.08x0.95mm_HandSolder -> Capacitor_SMD:C_0402_1005Metric_Pad0.74x0.62mm_HandSolder; Descr 100nF ±10% 50V X7R 0603 Multilayer Ceramic Capacitors MLCC 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 -> 100nF ±10% 16V X7R 0402 Multilayer Ceramic Capacitors MLCC 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; LCSC C14663 -> C1525
- C21: renamed from C19; value 22uF -> 10uF; footprint Capacitor_SMD:C_0603_1608Metric_Pad1.08x0.95mm_HandSolder -> Capacitor_SMD:C_0402_1005Metric_Pad0.74x0.62mm_HandSolder; Descr 22uF ±20% 6.3V X5R 0603 Multilayer Ceramic Capacitors MLCC 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 -> 10uF ±20% 6.3V X5R 0402 Multilayer Ceramic Capacitors MLCC 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; LCSC C59461 -> C15525
- C22: renamed from C20; value 22uF -> 10uF; footprint Capacitor_SMD:C_0603_1608Metric_Pad1.08x0.95mm_HandSolder -> Capacitor_SMD:C_0402_1005Metric_Pad0.74x0.62mm_HandSolder; Descr 22uF ±20% 6.3V X5R 0603 Multilayer Ceramic Capacitors MLCC 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 -> 10uF ±20% 6.3V X5R 0402 Multilayer Ceramic Capacitors MLCC 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; LCSC C59461 -> C15525
- C23: renamed from C21; footprint Capacitor_SMD:C_0603_1608Metric_Pad1.08x0.95mm_HandSolder -> Capacitor_SMD:C_0402_1005Metric_Pad0.74x0.62mm_HandSolder; Descr 100nF ±10% 50V X7R 0603 Multilayer Ceramic Capacitors MLCC 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 -> 100nF ±10% 16V X7R 0402 Multilayer Ceramic Capacitors MLCC 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; LCSC C14663 -> C1525
- C27: renamed from C22; footprint Capacitor_SMD:C_0603_1608Metric_Pad1.08x0.95mm_HandSolder -> Capacitor_SMD:C_0402_1005Metric_Pad0.74x0.62mm_HandSolder; Descr 100nF ±10% 50V X7R 0603 Multilayer Ceramic Capacitors MLCC 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 -> 100nF ±10% 16V X7R 0402 Multilayer Ceramic Capacitors MLCC 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; LCSC C14663 -> C1525
- C7: renamed from C5; footprint Capacitor_SMD:C_0603_1608Metric_Pad1.08x0.95mm_HandSolder -> Capacitor_SMD:C_0402_1005Metric_Pad0.74x0.62mm_HandSolder; Descr 100nF ±10% 50V X7R 0603 Multilayer Ceramic Capacitors MLCC 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 -> 100nF ±10% 16V X7R 0402 Multilayer Ceramic Capacitors MLCC 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; LCSC C14663 -> C1525
- C8: renamed from C6; footprint Capacitor_SMD:C_0603_1608Metric_Pad1.08x0.95mm_HandSolder -> Capacitor_SMD:C_0402_1005Metric_Pad0.74x0.62mm_HandSolder; Descr 470nF ±10% 25V X7R 0603 Multilayer Ceramic Capacitors MLCC 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 -> 470nF ±10% 10V X5R 0402 Multilayer Ceramic Capacitors MLCC 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; LCSC C1623 -> C47339
- C9: renamed from C7; footprint Capacitor_SMD:C_0603_1608Metric_Pad1.08x0.95mm_HandSolder -> Capacitor_SMD:C_0402_1005Metric_Pad0.74x0.62mm_HandSolder; Descr 100nF ±10% 50V X7R 0603 Multilayer Ceramic Capacitors MLCC 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 -> 100nF ±10% 16V X7R 0402 Multilayer Ceramic Capacitors MLCC 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; LCSC C14663 -> C1525
- J2: footprint Connector_PinHeader_1.27mm:PinHeader_2x05_P1.27mm_Vertical_SMD -> lib:PinHeader_2x05_P1.27mm_Vertical_SMD_case
- R1, R11, R9: footprint Resistor_SMD:R_0603_1608Metric_Pad0.98x0.95mm_HandSolder -> Resistor_SMD:R_0402_1005Metric_Pad0.72x0.64mm_HandSolder; Descr Chip Resistor - Surface Mount 100KOhms ±1% 1/10W 0603 RoHS -> 100kΩ ±1% 1/16W ±100ppm/℃ 0402 Chip Resistor - Surface Moun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; LCSC C25803 -> C25741
- R10, R5: footprint Resistor_SMD:R_0603_1608Metric_Pad0.98x0.95mm_HandSolder -> Resistor_SMD:R_0402_1005Metric_Pad0.72x0.64mm_HandSolder; Descr 1kΩ ±1% 0.1W ±100ppm/℃ 0603 Chip Resistor - Surface Mount R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 -> 1kΩ ±1% 1/16W ±100ppm/℃ 0402 Chip Resistor - Surface Mount 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; LCSC C21190 -> C11702
- R12, R6: footprint Resistor_SMD:R_0603_1608Metric_Pad0.98x0.95mm_HandSolder -> Resistor_SMD:R_0402_1005Metric_Pad0.72x0.64mm_HandSolder; Descr 47kΩ ±1% 0.1W ±100ppm/℃ 0603 Chip Resistor - Surface Mount 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 -> 47kΩ ±1% 1/16W ±100ppm/℃ 0402 Chip Resistor - Surface Mount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; LCSC C25819 -> C25792
- R13, R14: footprint Resistor_SMD:R_0603_1608Metric_Pad0.98x0.95mm_HandSolder -> Resistor_SMD:R_0402_1005Metric_Pad0.72x0.64mm_HandSolder; Descr 4.7K ±5% 1/10W ±100ppm/°C 0603 Chip Resistor - Surface Moun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 -> Chip Resistor - Surface Mount 4.7KOhms ±1% 1/16W 0402 RoHS; LCSC C105428 -> C25900
- R2: footprint Resistor_SMD:R_0603_1608Metric_Pad0.98x0.95mm_HandSolder -> Resistor_SMD:R_0402_1005Metric_Pad0.72x0.64mm_HandSolder; Descr 1.5kΩ ±1% 0.1W ±100ppm/℃ 0603 Chip Resistor - Surface Mount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 -> 1.5kΩ ±1% 1/16W ±100ppm/℃ 0402 Chip Resistor - Surface Moun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; LCSC C22843 -> C25867
- R3, R4: footprint Resistor_SMD:R_0603_1608Metric_Pad0.98x0.95mm_HandSolder -> Resistor_SMD:R_0402_1005Metric_Pad0.72x0.64mm_HandSolder; Descr 22Ω ±1% 0.1W ±200ppm/℃ 0603 Chip Resistor - Surface Mount R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 -> 22Ω ±1% 1/16W ±200ppm/℃ 0402 Chip Resistor - Surface Mount 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; LCSC C23345 -> C25092
- R7: footprint Resistor_SMD:R_0603_1608Metric_Pad0.98x0.95mm_HandSolder -> Resistor_SMD:R_0402_1005Metric_Pad0.72x0.64mm_HandSolder; Descr 100Ω ±1% 1/10W ±200ppm/°C 0603 Chip Resistor - Surface Moun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 -> 100Ω ±1% 1/16W ±200ppm/℃ 0402 Chip Resistor - Surface Mount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; LCSC C22775 -> C25076
- R8: footprint Resistor_SMD:R_0603_1608Metric_Pad0.98x0.95mm_HandSolder -> Resistor_SMD:R_0402_1005Metric_Pad0.72x0.64mm_HandSolder; Descr 2kΩ ±1% 0.1W ±100ppm/℃ 0603 Chip Resistor - Surface Mount R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 -> 2kΩ ±1% 1/16W ±100ppm/℃ 0402 Chip Resistor - Surface Mount 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; LCSC C22975 -> C4109
- renumbered C4 to C6, RN2 to RN1, RN3 to RN2
Connections:
- net labels added: E_USB+, E_USB-, USB+, USB-
- net labels removed: USBM, USBP
- wire segments 276 -> 299
- no-connect marks 23 -> 19
Other:
- moved on the sheet: R1, R2, R3, R4

Commit message: Version 2 of Normal PCB
Parts:
- removed R6: 47K, Resistor_SMD:R_0402_1005Metric_Pad0.72x0.64mm_HandSolder, symbol Device:R
- removed U4: LM358DR2G, Package_SO:SOIC-8_3.9x4.9mm_P1.27mm, symbol Amplifier_Operational:LM358
- added F1: Polyfuse, Fuse:Fuse_0603_1608Metric_Pad1.05x0.95mm_HandSolder, symbol Device:Polyfuse
- added JP1: VCC_SEL, Jumper:SolderJumper-3_P1.3mm_Bridged12_RoundedPad1.0x1.5mm, symbol Jumper:SolderJumper_3_Bridged12
- added U3: AD8531ARTZ, Package_TO_SOT_SMD:SOT-23-5_HandSoldering, symbol AD8531ARTZ-REEL7:AD8531ARTZ
- RN1: renamed from RN2; footprint Resistor_SMD:R_Array_Convex_4x0402 -> lib:R_Array_Convex_4x0402_hand_soldered
- RN2: renamed from RN1; footprint Resistor_SMD:R_Array_Convex_4x0402 -> lib:R_Array_Convex_4x0402_hand_soldered
- renumbered C9 to C10, C10 to C11, C11 to C12, C20 to C13, C12 to C14, C13 to C15, C21 to C16, C14 to C17, C22 to C18, C15 to C19, C23 to C20, C18 to C21, C19 to C22, C17 to C23, C16 to C8, C8 to C9, R15 to R12, R14 to R13, R13 to R14, R16 to R15, R7 to R6, R12 to R7, U3 to U4
Connections:
- net labels added: LRST, LRXD, LTCK, LTDI, LTDO, LTEST, LTMS, LTXD, VCC_OUT
- net labels removed: BRXD, BTXD, JENA
- wire segments 299 -> 293
- no-connect marks 19 -> 20
Other:
- moved on the sheet: C13, C16, C18, C20, C21, C22, C23, C24, C25, C26, C27, C8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

Commit message: Hardware V2 improvements (component values and sizes, layout and review of V-Target circuitry).
Parts:
- added C22: 10uF, Capacitor_SMD:C_0603_1608Metric_Pad1.08x0.95mm_HandSolder, symbol Device:C
- added C23: 100nF, Capacitor_SMD:C_0402_1005Metric_Pad0.74x0.62mm_HandSolder, symbol Device:C
- added R10: 4k7, Resistor_SMD:R_0402_1005Metric_Pad0.72x0.64mm_HandSolder, symbol Device:R
- J4: renamed from J5; footprint Connector_PinHeader_2.54mm:PinHeader_1x05_P2.54mm_Vertical -> Connector_PinHeader_2.54mm:PinHeader_1x06_P2.54mm_Vertical; symbol Connector:Conn_01x05_Male -> Connector:Conn_01x06_Male; Descr Pin Header 5 1 right-angle，180degrees 2.54mm Through Hole P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 -> Pin Header 6 1 right-angle，180degrees 2.54mm Through Hole P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
- U1: footprint Package_TO_SOT_SMD:SOT-223-3_TabPin2 -> Package_TO_SOT_SMD:SOT-89-3_Handsoldering; Descr Fixed 15V 3.3V 1.3V @ 800mA SOT-223 Dropout Regulators(LDO)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 -> Fixed 10V 3.3V 1.3V @ 1A SOT-89 Dropout Regulators(LDO) RoHS; LCSC C6186 -> C347256
- renumbered C14 to C13, C15 to C14, C17 to C15, C13 to C16, C19 to C17, C16 to C18, C18 to C19, C23 to C21, C21 to C28, C22 to C29, J4 to J3, J3 to J5, R8 to R11, R9 to R12, R10 to R13, R11 to R14, R12 to R15, R15 to R16, R13 to R5, R14 to R6, R5 to R7, R6 to R8, R7 to R9, RN2 to RN1, RN1 to RN2
Connections:
- wire segments 293 -> 310
Other:
- moved on the sheet: C16, C18, C19, C20, C21, C24, C25, C26, C27, C28, C29, C8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
