File: Hardware/Target_Proto_Boards/MSP_Proto/MSP_Proto.kicad_pcb (KiCad board)
At the start: 2 copper layers, 70 x 40 mm, 48 parts, among them J1 JTAG/SBW, J10 PORT6, J11 VCC, J12 GND, J13 +5V, J14 GND, J15 AVCC, J16 AGND, J2 VSEL, J3 LED_P4.1, J4 USB_B_Micro, J5 PORT1, J6 PORT2, J7 PORT3, J8 PORT4, J9 PORT5, SW1 TL-2203, U1 MSP430F2416TPM, U2 MSP430G2955IDA38, U3 HT7533-1, Y1 32768 12pF, Y2 16MHz

Commit message: Documentation for the MSP Proto board
Parts:
- added R6: 3.3k, Resistor_SMD:R_0603_1608Metric_Pad0.98x0.95mm_HandSolder, F.Cu at (124.4, 97.5)
- C3: value 1nF -> 2.2nF
- R1: value 470K -> 47K
- R2: value 470K -> 100K
Connections:
- C3 pad 1: /TDO -> Net-(C3-Pad1)
- R1 pad 2: /TDO -> Net-(C3-Pad1)
Routing:
- net +3V3: track 109.3 -> 104.9 mm
- net Net-(C3-Pad1): track 0.00 -> 3.73 mm
- net /TDO: track 28.8 -> 30.7 mm
Changed lines of the file:
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@@
-(kicad_pcb (version 20171130) (host pcbnew "(5.1.10)-1")
+(kicad_pcb (version 20171130) (host pcbnew "(5.1.12)-1")
   (general
     (thickness 1.6)
     (drawings 34)
-    (tracks 1134)
+    (tracks 1133)
     (zones 0)
-    (modules 48)
-    (nets 77)
+    (modules 49)
+    (nets 78)
   )
   (page A4)
   (layers
-    (0 F.Cu signal)
-    (31 B.Cu signal)
-    (33 F.Adhes user)
+    (0 F.Cu signal hide)
+    (31 B.Cu signal hide)
+    (33 F.Adhes user hide)
     (35 F.Paste user)
     (37 F.SilkS user)
@@
   (net 75 "Net-(SW1-Pad4)")
   (net 76 "Net-(SW1-Pad1)")
+  (net 77 "Net-(C3-Pad1)")
   (net_class Default "This is the default net class."
     (clearance 0.15)
@@
     (add_net /XT2IN)
     (add_net /XT2OUT)
+    (add_net "Net-(C3-Pad1)")
     (add_net "Net-(C5-Pad1)")
     (add_net "Net-(D1-Pad1)")
@@
     (add_net GNDA)
   )
+  (module Resistor_SMD:R_0603_1608Metric_Pad0.98x0.95mm_HandSolder (layer F.Cu)
+    (at 124.4 97.45 90)
+    (descr "Resistor SMD 0603 (1608 Metric), square (rectangular) end terminal, IPC_7351 nominal with elongated pad for handsoldering. (Body size source: IPC-SM-782 page 72, https://www.pcb-3d.com/wordpress/wp-content/uploads/ipc-sm-782a_amendment_1_and_2.pdf), generated with kicad-footprint-generator")
+    (tags "resistor handsolder")
+    (attr smd)
+    (fp_text reference R6 (at 2.35 0 90) (layer F.SilkS)
+      (effects (font (size 1 1) (thickness 0.15)))
+    )
+    (fp_text value 3.3k (at 0 1.43 90) (layer F.Fab)
+      (effects (font (size 1 1) (thickness 0.15)))
+    )
+    (fp_line (start 1.65 0.73) (end -1.65 0.73) (layer F.CrtYd) (width 0.05))
+    (fp_line (start 1.65 -0.73) (end 1.65 0.73) (layer F.CrtYd) (width 0.05))
+    (fp_line (start -1.65 -0.73) (end 1.65 -0.73) (layer F.CrtYd) (width 0.05))
+    (fp_line (start -1.65 0.73) (end -1.65 -0.73) (layer F.CrtYd) (width 0.05))
+    (fp_line (start -0.254724 0.5225) (end 0.254724 0.5225) (layer F.SilkS) (width 0.12))
+    (fp_line (start -0.254724 -0.5225) (end 0.254724 -0.5225) (layer F.SilkS) (width 0.12))
+    (fp_line (start 0.8 0.4125) (end -0.8 0.4125) (layer F.Fab) (width 0.1))
+    (fp_line (start 0.8 -0.4125) (end 0.8 0.4125) (layer F.Fab) (width 0.1))
+    (fp_line (start -0.8 -0.4125) (end 0.8 -0.4125) (layer F.Fab) (width 0.1))
+    (fp_line (start -0.8 0.4125) (end -0.8 -0.4125) (layer F.Fab) (width 0.1))
+    (fp_text user %R (at 0 0 90) (layer F.Fab)
+      (effects (font (size 0.4 0.4) (thickness 0.06)))
+    )
+    (pad 2 smd roundrect (at 0.9125 0 90) (size 0.975 0.95) (layers F.Cu F.Paste F.Mask) (roundrect_rratio 0.25)
+      (net 2 /TDO))
+    (pad 1 smd roundrect (at -0.9125 0 90) (size 0.975 0.95) (layers F.Cu F.Paste F.Mask) (roundrect_rratio 0.25)
+      (net 77 "Net-(C3-Pad1)"))
+    (model ${KISYS3DMOD}/Resistor_SMD.3dshapes/R_0603_1608Metric.wrl
+      (at (xyz 0 0 0))
+      (scale (xyz 1 1 1))
+      (rotate (xyz 0 0 0))
+    )
+  )
   (module Crystal:Crystal_SMD_3225-4Pin_3.2x2.5mm_HandSoldering (layer F.Cu)
     (at 129.1 97.65 270)
@@
     (tags "Micro-USB SMD Typ-B")
     (attr smd)
-    (fp_text reference J4 (at 0 -3.1125 90) (layer F.SilkS)
+    (fp_text reference J4 (at 4.95 -0.01 180) (layer F.SilkS)
       (effects (font (size 1 1) (thickness 0.15)))
     )
@@
     (tags "resistor handsolder")
     (attr smd)
-    (fp_text reference R2 (at 0 1.2 90) (layer F.SilkS)
+    (fp_text reference R2 (at -2.35 0 90) (layer F.SilkS)
       (effects (font (size 1 1) (thickness 0.15)))
     )
-    (fp_text value 470K (at 0 1.43 90) (layer F.Fab)
+    (fp_text value 100K (at 0 1.43 90) (layer F.Fab)
       (effects (font (size 1 1) (thickness 0.15)))
     )
@@
     (tags "resistor handsolder")
     (attr smd)
-    (fp_text reference R1 (at 0 -1.3 90) (layer F.SilkS)
+    (fp_text reference R1 (at -2.35 0 90) (layer F.SilkS)
       (effects (font (size 1 1) (thickness 0.15)))
     )
-    (fp_text value 470K (at 0 1.43 90) (layer F.Fab)
+    (fp_text value 47K (at 0 1.43 90) (layer F.Fab)
       (effects (font (size 1 1) (thickness 0.15)))
     )
@@
     )
     (pad 2 smd roundrect (at 0.9125 0 270) (size 0.975 0.95) (layers F.Cu F.Paste F.Mask) (roundrect_rratio 0.25)
-      (net 2 /TDO))
+      (net 77 "Net-(C3-Pad1)"))
     (pad 1 smd roundrect (at -0.9125 0 270) (size 0.975 0.95) (layers F.Cu F.Paste F.Mask) (roundrect_rratio 0.25)
       (net 10 +3V3))
@@
       (effects (font (size 1 1) (thickness 0.15)))
     )
-    (fp_text value 1nF (at 0 1.43 90) (layer F.Fab)
+    (fp_text value 2.2nF (at 0 1.43 90) (layer F.Fab)
       (effects (font (size 1 1) (thickness 0.15)))
     )
@@
       (net 1 GND))
     (pad 1 smd roundrect (at -0.8625 0 270) (size 1.075 0.95) (layers F.Cu F.Paste F.Mask) (roundrect_rratio 0.25)
-      (net 2 /TDO))
+      (net 77 "Net-(C3-Pad1)"))
     (model ${KISYS3DMOD}/Capacitor_SMD.3dshapes/C_0603_1608Metric.wrl
       (at (xyz 0 0 0))
@@
   (segment (start 134.1 104.2) (end 134.1 105) (width 0.2) (layer B.Cu) (net 2))
   (segment (start 132.15 102.25) (end 134.1 104.2) (width 0.2) (layer B.Cu) (net 2))
-  (segment (start 122.9 100.5875) (end 122.9 98.3625) (width 0.2) (layer F.Cu) (net 2))
-  (segment (start 121.86251 97.32501) (end 122.9 98.3625) (width 0.2) (layer F.Cu) (net 2))
-  (segment (start 114.77501 97.32501) (end 121.86251 97.32501) (width 0.2) (layer F.Cu) (net 2))
+  (segment (start 123.61249 97.32501) (end 124.4 96.5375) (width 0.2) (layer F.Cu) (net 2))
+  (segment (start 114.77501 97.32501) (end 123.61249 97.32501) (width 0.2) (layer F.Cu) (net 2))
   (segment (start 113.4 95.95) (end 114.77501 97.32501) (width 0.2) (layer F.Cu) (net 2))
-  (segment (start 125.7 102.25) (end 132.15 102.25) (width 0.2) (layer F.Cu) (net 2))
-  (segment (start 124.0375 100.5875) (end 125.7 102.25) (width 0.2) (layer F.Cu) (net 2))
-  (segment (start 122.9 100.5875) (end 124.0375 100.5875) (width 0.2) (layer F.Cu) (net 2))
+  (segment (start 125.12501 101.72501) (end 125.12501 97.26251) (width 0.2) (layer F.Cu) (net 2))
+  (segment (start 125.12501 97.26251) (end 124.4 96.5375) (width 0.2) (layer F.Cu) (net 2))
+  (segment (start 125.65 102.25) (end 125.12501 101.72501) (width 0.2) (layer F.Cu) (net 2))
+  (segment (start 132.15 102.25) (end 125.65 102.25) (width 0.2) (layer F.Cu) (net 2))
   (segment (start 130.21099 104.25) (end 129.960979 104.500011) (width 0.2) (layer F.Cu) (net 3))
   (segment (start 133.325 104.25) (end 130.21099 104.25) (width 0.2) (layer F.Cu) (net 3))
@@
   (segment (start 117.913012 101.37501) (end 116.128003 99.590001) (width 0.2) (layer F.Cu) (net 9))
   (segment (start 123.67501 101.37501) (end 117.913012 101.37501) (width 0.2) (layer F.Cu) (net 9))
-  (segment (start 125.05 102.75) (end 123.67501 101.37501) (width 0.2) (layer F.Cu) (net 9))
+  (segment (start 123.67501 101.37501) (end 125.05 102.75) (width 0.2) (layer F.Cu) (net 9))
   (via (at 133.8 108.7) (size 0.6) (drill 0.3) (layers F.Cu B.Cu) (net 10))
   (segment (start 135.2875 108.7) (end 133.8 108.7) (width 0.254) (layer B.Cu) (net 10))
@@
   (segment (start 127.35 96.6) (end 127.419999 96.669999) (width 0.508) (layer B.Cu) (net 10))
   (segment (start 127.419999 96.669999) (end 127.419999 103.069999) (width 1) (layer B.Cu) (net 10))
-  (via (at 124.3 96.55) (size 0.6) (drill 0.3) (layers F.Cu B.Cu) (net 10))
+  (via (at 122.9 95.35) (size 0.6) (drill 0.3) (layers F.Cu B.Cu) (net 10))
   (segment (start 121.4 96.5375) (end 122.9 96.5375) (width 0.387) (layer F.Cu) (net 10))
-  (segment (start 124.2875 96.5375) (end 124.3 96.55) (width 0.387) (layer F.Cu) (net 10))
-  (segment (start 122.9 96.5375) (end 124.2875 96.5375) (width 0.387) (layer F.Cu) (net 10))
   (segment (start 127.419999 94.479999) (end 127.419999 96.669999) (width 1) (layer B.Cu) (net 10))
   (segment (start 123.99 91.05) (end 127.419999 94.479999) (width 1) (layer B.Cu) (net 10))
   (segment (start 127.3 96.55) (end 127.419999 96.669999) (width 0.381) (layer B.Cu) (net 10))
-  (segment (start 124.3 96.55) (end 127.3 96.55) (width 0.381) (layer B.Cu) (net 10))
   (segment (start 145.85 113.1) (end 132.1 113.1) (width 1) (layer B.Cu) (net 10))
   (segment (start 153.1 103.8625) (end 151.6 103.8625) (width 0.75) (layer F.Cu) (net 10))
@@
   (segment (start 172.76 104.25) (end 171.05 104.25) (width 0.381) (layer F.Cu) (net 74))
   (segment (start 169.85 103.05) (end 165.35 103.05) (width 0.75) (layer F.Cu) (net 74))
+  (segment (start 122.9 100.5875) (end 122.9 98.3625) (width 0.2) (layer F.Cu) (net 77))
+  (segment (start 122.9 98.3625) (end 124.4 98.3625) (width 0.2) (layer F.Cu) (net 77))
   (zone (net 1) (net_name GND) (layer F.Cu) (hatch edge 0.508)
     (connect_pads (clearance 0.508))
