File: Hardware/Target_Proto_Boards/MSP_Proto/MSP_Proto.sch (KiCad schematic (older format))
At the start: 48 parts, among them J1 JTAG/SBW, J10 PORT6, J11 VCC, J12 GND, J13 +5V, J14 GND, J15 AVCC, J16 AGND, J2 VSEL, J3 LED_P4.1, J4 USB_B_Micro, J5 PORT1, J6 PORT2, J7 PORT3, J8 PORT4, J9 PORT5, SW1 TL-2203, U1 MSP430F2416TPM, U2 MSP430G2955IDA38, U3 HT7533-1, Y1 32768 12pF, Y2 16MHz

Commit message: Documentation for the MSP Proto board
Parts:
- added R6: 3.3k, Resistor_SMD:R_0603_1608Metric_Pad0.98x0.95mm_HandSolder, symbol Device:R
- C3: value 1nF -> 2.2nF; Descr 0603 Multilayer Ceramic Capacitors MLCC - SMD/SMT ROHS -> X7R 2.2nF ±10% 50V 0603 Multilayer Ceramic Capacitors MLCC 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; LCSC C1588 -> C1604
- R1: value 470K -> 47K; Descr 0603 Chip Resistor - Surface Mount ROHS -> ±1% ±100ppm/℃ 0.1W 47kΩ 0603 Chip Resistor - Surface Mount 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; LCSC C23178 -> C25819
- R2: value 470K -> 100K; Descr 0603 Chip Resistor - Surface Mount ROHS -> ±1% 100kΩ ±100ppm/℃ 0.1W 0603 Chip Resistor - Surface Mount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; LCSC C23178 -> C25803
Connections:
- net TDO: now also R6.2; no longer C3.1, R1.2
- new net: C3.1, R1.2, R6.1
Other:
- moved on the sheet: C3, C7, R1, R2
Changed lines of the file:
@@
 L Device:R R2
 U 1 1 61050AC2
-P 1900 5900
-F 0 "R2" H 1970 5946 50  0000 L CNN
-F 1 "470K" H 1970 5855 50  0000 L CNN
-F 2 "Resistor_SMD:R_0603_1608Metric_Pad0.98x0.95mm_HandSolder" V 1830 5900 50  0001 C CNN
-F 3 "~" H 1900 5900 50  0001 C CNN
-F 4 "0603 Chip Resistor - Surface Mount ROHS" H 1900 5900 50  0001 C CNN "Descr"
-F 5 "C23178" H 1900 5900 50  0001 C CNN "LCSC"
-	1    1900 5900
+P 1900 5950
+F 0 "R2" H 1970 5996 50  0000 L CNN
+F 1 "100K" H 1970 5905 50  0000 L CNN
+F 2 "Resistor_SMD:R_0603_1608Metric_Pad0.98x0.95mm_HandSolder" V 1830 5950 50  0001 C CNN
+F 3 "~" H 1900 5950 50  0001 C CNN
+F 4 "±1% 100kΩ ±100ppm/℃ 0.1W 0603 Chip Resistor - Surface Mount ROHS" H 1900 5950 50  0001 C CNN "Descr"
+F 5 "C25803" H 1900 5950 50  0001 C CNN "LCSC"
+	1    1900 5950
 	1    0    0    -1
 $EndComp
@@
 L Device:C C7
 U 1 1 61052779
-P 1900 6300
-F 0 "C7" H 2015 6346 50  0000 L CNN
-F 1 "47nF" H 2015 6255 50  0000 L CNN
-F 2 "Capacitor_SMD:C_0603_1608Metric_Pad1.08x0.95mm_HandSolder" H 1938 6150 50  0001 C CNN
-F 3 "~" H 1900 6300 50  0001 C CNN
-F 4 "C1622" H 1900 6300 50  0001 C CNN "LCSC"
-F 5 "0603 Multilayer Ceramic Capacitors MLCC - SMD/SMT ROHS" H 1900 6300 50  0001 C CNN "Descr"
-	1    1900 6300
+P 1900 6350
+F 0 "C7" H 2015 6396 50  0000 L CNN
+F 1 "47nF" H 2015 6305 50  0000 L CNN
+F 2 "Capacitor_SMD:C_0603_1608Metric_Pad1.08x0.95mm_HandSolder" H 1938 6200 50  0001 C CNN
+F 3 "~" H 1900 6350 50  0001 C CNN
+F 4 "C1622" H 1900 6350 50  0001 C CNN "LCSC"
+F 5 "0603 Multilayer Ceramic Capacitors MLCC - SMD/SMT ROHS" H 1900 6350 50  0001 C CNN "Descr"
+	1    1900 6350
 	1    0    0    -1
 $EndComp
@@
 	2500 5950 2250 5950
 Wire Wire Line
-	2250 5950 2250 6100
+	2250 5950 2250 6150
 $Comp
 L power:GND #PWR010
 U 1 1 61053FF5
-P 1900 6500
-F 0 "#PWR010" H 1900 6250 50  0001 C CNN
-F 1 "GND" H 1905 6327 50  0000 C CNN
-F 2 "" H 1900 6500 50  0001 C CNN
-F 3 "" H 1900 6500 50  0001 C CNN
-	1    1900 6500
+P 1900 6550
+F 0 "#PWR010" H 1900 6300 50  0001 C CNN
+F 1 "GND" H 1905 6377 50  0000 C CNN
+F 2 "" H 1900 6550 50  0001 C CNN
+F 3 "" H 1900 6550 50  0001 C CNN
+	1    1900 6550
 	1    0    0    -1
 $EndComp
@@
 L power:+3.3V #PWR09
 U 1 1 610545AB
-P 1900 5700
-F 0 "#PWR09" H 1900 5550 50  0001 C CNN
-F 1 "+3.3V" H 1915 5873 50  0000 C CNN
-F 2 "" H 1900 5700 50  0001 C CNN
-F 3 "" H 1900 5700 50  0001 C CNN
-	1    1900 5700
-	1    0    0    -1
-$EndComp
-Wire Wire Line
-	1900 5750 1900 5700
+P 1900 5750
+F 0 "#PWR09" H 1900 5600 50  0001 C CNN
+F 1 "+3.3V" H 1915 5923 50  0000 C CNN
+F 2 "" H 1900 5750 50  0001 C CNN
+F 3 "" H 1900 5750 50  0001 C CNN
+	1    1900 5750
+	1    0    0    -1
+$EndComp
+Wire Wire Line
+	1900 5800 1900 5750
 Text Label 2250 5950 0    50   ~ 0
 RESET
@@
 TDO
 Wire Wire Line
-	1900 6450 1900 6500
+	1900 6500 1900 6550
 $Comp
 L Device:R R1
 U 1 1 610A259C
-P 1450 5250
-F 0 "R1" H 1520 5296 50  0000 L CNN
-F 1 "470K" H 1520 5205 50  0000 L CNN
-F 2 "Resistor_SMD:R_0603_1608Metric_Pad0.98x0.95mm_HandSolder" V 1380 5250 50  0001 C CNN
-F 3 "~" H 1450 5250 50  0001 C CNN
-F 4 "0603 Chip Resistor - Surface Mount ROHS" H 1450 5250 50  0001 C CNN "Descr"
-F 5 "C23178" H 1450 5250 50  0001 C CNN "LCSC"
-	1    1450 5250
+P 1250 5250
+F 0 "R1" H 1320 5296 50  0000 L CNN
+F 1 "47K" H 1320 5205 50  0000 L CNN
+F 2 "Resistor_SMD:R_0603_1608Metric_Pad0.98x0.95mm_HandSolder" V 1180 5250 50  0001 C CNN
+F 3 "~" H 1250 5250 50  0001 C CNN
+F 4 "±1% ±100ppm/℃ 0.1W 47kΩ 0603 Chip Resistor - Surface Mount ROHS" H 1250 5250 50  0001 C CNN "Descr"
+F 5 "C25819" H 1250 5250 50  0001 C CNN "LCSC"
+	1    1250 5250
 	1    0    0    -1
 $EndComp
@@
 L Device:C C3
 U 1 1 610A2A4A
-P 1450 5650
-F 0 "C3" H 1565 5696 50  0000 L CNN
-F 1 "1nF" H 1565 5605 50  0000 L CNN
-F 2 "Capacitor_SMD:C_0603_1608Metric_Pad1.08x0.95mm_HandSolder" H 1488 5500 50  0001 C CNN
-F 3 "~" H 1450 5650 50  0001 C CNN
-F 4 "0603 Multilayer Ceramic Capacitors MLCC - SMD/SMT ROHS" H 1450 5650 50  0001 C CNN "Descr"
-F 5 "C1588" H 1450 5650 50  0001 C CNN "LCSC"
-	1    1450 5650
+P 1250 5650
+F 0 "C3" H 1365 5696 50  0000 L CNN
+F 1 "2.2nF" H 1365 5605 50  0000 L CNN
+F 2 "Capacitor_SMD:C_0603_1608Metric_Pad1.08x0.95mm_HandSolder" H 1288 5500 50  0001 C CNN
+F 3 "~" H 1250 5650 50  0001 C CNN
+F 4 "X7R 2.2nF ±10% 50V 0603 Multilayer Ceramic Capacitors MLCC - SMD/SMT ROHS" H 1250 5650 50  0001 C CNN "Descr"
+F 5 "C1604" H 1250 5650 50  0001 C CNN "LCSC"
+	1    1250 5650
 	1    0    0    -1
 $EndComp
@@
 L power:+3.3V #PWR04
 U 1 1 610A3AAB
-P 1450 5050
-F 0 "#PWR04" H 1450 4900 50  0001 C CNN
-F 1 "+3.3V" H 1465 5223 50  0000 C CNN
-F 2 "" H 1450 5050 50  0001 C CNN
-F 3 "" H 1450 5050 50  0001 C CNN
-	1    1450 5050
+P 1250 5050
+F 0 "#PWR04" H 1250 4900 50  0001 C CNN
+F 1 "+3.3V" H 1265 5223 50  0000 C CNN
+F 2 "" H 1250 5050 50  0001 C CNN
+F 3 "" H 1250 5050 50  0001 C CNN
+	1    1250 5050
 	1    0    0    -1
 $EndComp
@@
 L power:GND #PWR05
 U 1 1 610A3FC7
-P 1450 5850
-F 0 "#PWR05" H 1450 5600 50  0001 C CNN
-F 1 "GND" H 1455 5677 50  0000 C CNN
-F 2 "" H 1450 5850 50  0001 C CNN
-F 3 "" H 1450 5850 50  0001 C CNN
-	1    1450 5850
-	1    0    0    -1
-$EndComp
-Wire Wire Line
-	1450 5100 1450 5050
-Wire Wire Line
-	1450 5850 1450 5800
-Wire Wire Line
-	1900 6050 1900 6100
-Wire Wire Line
-	2250 6100 1900 6100
-Connection ~ 1900 6100
+P 1250 5850
+F 0 "#PWR05" H 1250 5600 50  0001 C CNN
+F 1 "GND" H 1255 5677 50  0000 C CNN
+F 2 "" H 1250 5850 50  0001 C CNN
+F 3 "" H 1250 5850 50  0001 C CNN
+	1    1250 5850
+	1    0    0    -1
+$EndComp
+Wire Wire Line
+	1250 5100 1250 5050
+Wire Wire Line
+	1250 5850 1250 5800
 Wire Wire Line
 	1900 6100 1900 6150
 Wire Wire Line
-	1450 5400 1450 5450
-Wire Wire Line
-	1450 5450 2500 5450
-Connection ~ 1450 5450
-Wire Wire Line
-	1450 5450 1450 5500
+	2250 6150 1900 6150
+Connection ~ 1900 6150
+Wire Wire Line
+	1900 6150 1900 6200
+Wire Wire Line
+	1250 5400 1250 5450
+Wire Wire Line
+	1250 5450 1450 5450
+Connection ~ 1250 5450
+Wire Wire Line
+	1250 5450 1250 5500
 Wire Wire Line
 	8800 3850 9100 3850
@@
 Wire Wire Line
 	1550 3950 1550 4500
+$Comp
+L Device:R R6
+U 1 1 61A82441
+P 1600 5450
+F 0 "R6" V 1700 5450 50  0000 C CNN
+F 1 "3.3k" V 1500 5450 50  0000 C CNN
+F 2 "Resistor_SMD:R_0603_1608Metric_Pad0.98x0.95mm_HandSolder" V 1530 5450 50  0001 C CNN
+F 3 "~" H 1600 5450 50  0001 C CNN
+F 4 "3.3kΩ ±1% ±100ppm/℃ 0.1W 0603 Chip Resistor - Surface Mount ROHS" H 1600 5450 50  0001 C CNN "Descr"
+F 5 "C22978" H 1600 5450 50  0001 C CNN "LCSC"
+	1    1600 5450
+	0    -1   -1   0
+$EndComp
+Wire Wire Line
+	1750 5450 2500 5450
 $EndSCHEMATC
