File: Hardware/Target_Proto_Boards/MSP_Proto/MSP_Proto.kicad_sch (KiCad schematic)
At the start: 49 parts, among them J1 JTAG/SBW, J10 PORT6, J11 VCC, J12 GND, J13 +5V, J14 GND, J15 AVCC, J16 AGND, J2 VSEL, J3 LED_P4.1, J4 USB_B_Micro, J5 PORT1, J6 PORT2, J7 PORT3, J8 PORT4, J9 PORT5, SW1 TL-2203, U1 MSP430F2416TPM, U2 MSP430G2955IDA38, U3 HT7533-1, Y1 32768 12pF, Y2 16MHz

Commit message: Missing changes for KiCad 6 migration
Parts:
- NT1: symbol MSP_Proto-rescue:Net-Tie_2-Device -> Device:NetTie_2
Changed lines of the file:
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@@
     (pin "1")
   )
-  (symbol (lib_id "MSP_Proto-rescue:Net-Tie_2-Device") (at 157.48 177.8 0) (unit 1)
+  (symbol (lib_id "Device:NetTie_2") (at 157.48 177.8 0) (unit 1)
     (in_bom yes) (on_board yes)
     (property "Reference" "NT1" (id 0) (at 157.48 173.2026 0))
