File: Hardware/Target_Proto_Boards/F5418/F5418.kicad_pcb (KiCad board)
At the start: 2 copper layers, 90 x 50 mm, 51 parts, among them J1 LED_P4.1, J10 PORT4, J11 PORT8, J12 JTAG/SBW, J13 VCC, J14 GND, J15 +5V, J16 GND, J17 VSEL, J18 LogAna, J19 AS, J2 PORT1, J3 PORT5, J4 DEBUG, J5 PORT2, J6 PORT6, J7 USB_B_Micro, J8 PORT3, J9 PORT7, SW1 RESET, SW2 TL-2203, U1 MSP430F5418IPNR, U2 HT7533-1, Y1 32768 12pF, Y2 25 MHz

Commit message: Updated Hardware Schematics and Boards
Parts:
- added R5: 3.3k, Resistor_SMD:R_0603_1608Metric_Pad0.98x0.95mm_HandSolder, F.Cu at (112.4, 115.0)
- added R6: 330, Resistor_SMD:R_0603_1608Metric_Pad0.98x0.95mm_HandSolder, F.Cu at (100.5, 108.7)
- C3: value 1nF -> 2.2nF
Connections:
- C3 pad 1: /RESET -> Net-(C3-Pad1)
- J4 pad 10: /JTEST -> Net-(J4-Pad10)
- R1 pad 2: /RESET -> Net-(C3-Pad1)
- SW1 pad 1: /RESET -> Net-(C3-Pad1)
Routing:
- net Net-(C3-Pad1): track 0.00 -> 10.7 mm
- net /RESET: track 48.7 -> 41.0 mm
- net Net-(J4-Pad10): track 0.00 -> 6.73 mm
- net /JTEST: track 46.0 -> 48.4 mm
- net +3V3: track 229.3 -> 231.0 mm
- net /JTXD: track 93.7 -> 92.8 mm
- net /JRST: track 17.9 -> 18.6 mm

Commit message: F5418 boarf updated to KiCad6
Other:
- net class Default removed
- net class Power removed
