File: Hardware/Target_Proto_Boards/SLAU208_F5418/F5418.kicad_sch (KiCad schematic)
At the start: 53 parts, among them J1 LED_P4.1, J10 PORT4, J11 PORT8, J12 JTAG/SBW, J13 VCC, J14 GND, J15 +5V, J16 GND, J17 VSEL, J18 LogAna, J19 AS, J2 PORT1, J3 PORT5, J4 DEBUG, J5 PORT2, J6 PORT6, J7 USB_B_Micro, J8 PORT3, J9 PORT7, SW1 RESET, SW2 TL-2203, U1 MSP430F5418IPNR, U2 HT7533-1, Y1 32768 12pF, Y2 25 MHz

Commit message: Updated SLAU208
Parts:
- removed C1, C19, C2, C20: 22pF, Capacitor_SMD:C_0603_1608Metric_Pad1.08x0.95mm_HandSolder, symbol Device:C
- C1: renamed from C3; Descr X7R 2.2nF ±10% 50V 0603 Multilayer Ceramic Capacitors MLCC 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 -> 50V 2.2nF X7R ±10% 0603 Multilayer Ceramic Capacitors MLCC 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
- C10: renamed from C21; Descr 0603 Multilayer Ceramic Capacitors MLCC - SMD/SMT ROHS -> 25V 220nF X7R ±10% 0603 Multilayer Ceramic Capacitors MLCC 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
- C11: renamed from C12; Descr 0603 Multilayer Ceramic Capacitors MLCC - SMD/SMT ROHS -> 25V 220nF X7R ±10% 0603 Multilayer Ceramic Capacitors MLCC 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
- C12: renamed from C17; Descr 0603 Multilayer Ceramic Capacitors MLCC - SMD/SMT ROHS -> 10V 10uF X5R ±10% 0603 Multilayer Ceramic Capacitors MLCC -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
- C13, C14: Descr 0603 Multilayer Ceramic Capacitors MLCC - SMD/SMT ROHS -> 25V 220nF X7R ±10% 0603 Multilayer Ceramic Capacitors MLCC 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
- C15: renamed from C18; Descr 0603 Multilayer Ceramic Capacitors MLCC - SMD/SMT ROHS -> 25V 220nF X7R ±10% 0603 Multilayer Ceramic Capacitors MLCC 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
- C16: renamed from C15; Descr 0603 Multilayer Ceramic Capacitors MLCC - SMD/SMT ROHS -> 10V 10uF X5R ±10% 0603 Multilayer Ceramic Capacitors MLCC -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
- C17: renamed from C16; Descr 0603 Multilayer Ceramic Capacitors MLCC - SMD/SMT ROHS -> 10V 10uF X5R ±10% 0603 Multilayer Ceramic Capacitors MLCC -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
- C2: renamed from C4; Descr 0603 Multilayer Ceramic Capacitors MLCC - SMD/SMT ROHS -> 10V 10uF X5R ±10% 0603 Multilayer Ceramic Capacitors MLCC -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
- C3: renamed from C5; Descr 0603 Multilayer Ceramic Capacitors MLCC - SMD/SMT ROHS -> 25V 220nF X7R ±10% 0603 Multilayer Ceramic Capacitors MLCC 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
- C4: renamed from C6; Descr 0603 Multilayer Ceramic Capacitors MLCC - SMD/SMT ROHS -> 25V 220nF X7R ±10% 0603 Multilayer Ceramic Capacitors MLCC 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
- C5: renamed from C7; Descr 0603 Multilayer Ceramic Capacitors MLCC - SMD/SMT ROHS -> 25V 220nF X7R ±10% 0603 Multilayer Ceramic Capacitors MLCC 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
- C6: renamed from C8; Descr 0603 Multilayer Ceramic Capacitors MLCC - SMD/SMT ROHS -> 25V 220nF X7R ±10% 0603 Multilayer Ceramic Capacitors MLCC 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
- C7: renamed from C9; Descr 0603 Multilayer Ceramic Capacitors MLCC - SMD/SMT ROHS -> 25V 220nF X7R ±10% 0603 Multilayer Ceramic Capacitors MLCC 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
- C8: renamed from C10; Descr X7R ±10% 50V 470nF 0805 Multilayer Ceramic Capacitors MLCC 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 -> 50V 470nF X7R ±10% 0805 Multilayer Ceramic Capacitors MLCC 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
- C9: renamed from C11; Descr 0603 Multilayer Ceramic Capacitors MLCC - SMD/SMT ROHS -> 10V 10uF X5R ±10% 0603 Multilayer Ceramic Capacitors MLCC -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
- J1: value LED_P4.1 -> LED4.1
- J10: renamed from J4; value DEBUG -> J/S
- J13: renamed from J12; value JTAG/SBW -> JTAG
- J14: renamed from J13; value VCC -> 3V3
- J16: renamed from J15; value +5V -> 5V
- J18: renamed from J19; value AS -> AVCC
- J19: renamed from J17; value VSEL -> VRef
- J4: renamed from J7; Descr 1 1A 母座 USB - Micro B 5 USB 2.0 SMD USB Connectors ROHS -> 1A USB 2.0 1 5 Female Micro-B SMD USB Connectors ROHS
- J5: renamed from J18; value LogAna -> LogicAna
- L1: renamed from R3; value 22 -> 1K8; footprint Resistor_SMD:R_0603_1608Metric_Pad0.98x0.95mm_HandSolder -> Inductor_SMD:L_0603_1608Metric_Pad1.05x0.95mm_HandSolder; symbol Device:R -> Device:L_Ferrite_Small; Descr ±1% ±200ppm/℃ 0.1W 22Ω 0603 Chip Resistor - Surface Mount R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 -> 200mA 1 850mΩ 1.8kΩ@100MHz ±25% 0603 Ferrite Beads ROHS; LCSC C23345 -> C279972
- NT1: renamed from R4; value 0R -> NetTie_2; footprint Resistor_SMD:R_0603_1608Metric_Pad0.98x0.95mm_HandSolder -> NetTie:NetTie-2_SMD_Pad0.5mm; symbol Device:R -> Device:NetTie_2; Descr - ±1% 0Ω 0.1W 0603 Chip Resistor - Surface Mount ROHS -> (none); LCSC C21189 -> (none)
- R1: Descr 0603 Chip Resistor - Surface Mount ROHS -> 100mW Thick Film Resistors 75V ±100ppm/℃ ±1% -55℃~+155℃ 47k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; LCSC (none) -> (none)
- R2: renamed from R5; value 3.3k -> 3K3; Descr 3.3kΩ ±1% ±100ppm/℃ 0.1W 0603 Chip Resistor - Surface Mount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 -> 100mW Thick Film Resistors 75V ±100ppm/℃ ±1% -55℃~+155℃ 3.3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
- R3: renamed from R2; Descr 0603 Chip Resistor - Surface Mount ROHS -> 100mW Thick Film Resistors 75V ±100ppm/℃ ±1% -55℃~+155℃ 1kΩ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
- R4: renamed from R6; Descr ±1% 330Ω ±100ppm/℃ 0.1W 0603 Chip Resistor - Surface Mount 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 -> 100mW Thick Film Resistors 75V ±100ppm/℃ ±1% -55℃~+155℃ 330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
- SW1: Descr SMD,3×4×2.0mm Tactile Switches ROHS -> O SMDSplicing 50mA 4mm 100MΩ 100000 12V 160gf@±50gf 3mm -30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
- U1: Descr (none) -> LQFP-80_12x12x05P Microcontroller Units (MCUs/MPUs/SOCs) RO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; LCSC (none) -> C59496
- U2: value HT7533-1 -> HT7333-A; footprint Package_TO_SOT_SMD:SOT-89-3_Handsoldering -> Package_TO_SOT_SMD:SOT-89-3; Descr SOT-89(SOT-89-3) Linear Voltage Regulators (LDO) ROHS -> 250mA 90mV@(40mA) Fixed 3.3V~3.3V Positive 1 12V SOT-89 Lin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; LCSC C14289 -> C347191
- Y1: renamed from Y2; value 25 MHz -> CSTNE24M0; footprint Crystal:Crystal_SMD_3225-4Pin_3.2x2.5mm_HandSoldering -> Crystal:Resonator_SMD_Murata_CSTxExxV-3Pin_3.0x1.1mm; symbol Device:Crystal_GND24_Small -> Device:Resonator_Small; Descr ±10ppm 12pF -40℃~85℃ 贴片无源晶振 40Ω 25000000Hz SMD3225-4P Cryst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 -> ±0.11% 20MHz 15pF 40Ω SMD3213-3P Ceramic Resonators ROHS; LCSC C9006 -> C2650766
- Y2: renamed from Y1; value 32768 12pF -> 32768; Descr SMD3215-2P Crystals ROHS -> 32.768kHz SMD Crystal Resonator 7pF 70kΩ ±20ppm -40℃~+85℃ S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; LCSC C32346 -> C48615
- renumbered J10 to J11, J11 to J12, J14 to J15, J16 to J17, J5 to J6, J6 to J7
Connections:
- net GND: no longer Y1.4
- net JRST: now also J5.6 (Pin_6)
- net JTCK: now also J5.1 (Pin_1)
- net JTDO: now also J5.4 (Pin_4)
- net RESET: no longer J5.6 (Pin_6)
- net TCK: no longer J5.1 (Pin_1)
- net TDO: no longer J5.4 (Pin_4)
- net +3V3 renamed +3.3V
Other:
- moved on the sheet: NT1
