File: Hardware/Target_Proto_Boards/SLAU208_F5418/F5418.kicad_pcb (KiCad board)
At the start: 2 copper layers, 90 x 50 mm, 53 parts, among them J1 LED_P4.1, J10 PORT4, J11 PORT8, J12 JTAG/SBW, J13 VCC, J14 GND, J15 +5V, J16 GND, J17 VSEL, J18 LogAna, J19 AS, J2 PORT1, J3 PORT5, J4 DEBUG, J5 PORT2, J6 PORT6, J7 USB_B_Micro, J8 PORT3, J9 PORT7, SW1 RESET, SW2 TL-2203, U1 MSP430F5418IPNR, U2 HT7533-1, Y1 32768 12pF, Y2 25 MHz

Commit message: Updated SLAU208
Parts:
- removed the C1 at (140.6, 120.5)
- removed C19, C20: 22pF, Capacitor_SMD:C_0603_1608Metric_Pad1.08x0.95mm_HandSolder
- removed the C2 at (137.2, 120.5)
- J1: value LED_P4.1 -> LED4.1
- J10: renamed from J4; value DEBUG -> J/S
- J13: renamed from J12; value JTAG/SBW -> JTAG
- J14: renamed from J13; value VCC -> 3V3
- J16: renamed from J15; value +5V -> 5V
- J18: renamed from J19; value AS -> AVCC
- J19: renamed from J17; value VSEL -> VRef
- J5: renamed from J18; value LogAna -> LogicAna
- L1: renamed from R3; value 22 -> 1K8; footprint Resistor_SMD:R_0603_1608Metric_Pad0.98x0.95mm_HandSolder -> Inductor_SMD:L_0603_1608Metric_Pad1.05x0.95mm_HandSolder
- NT1: renamed from R4; value 0R -> NetTie_2; footprint Resistor_SMD:R_0603_1608Metric_Pad0.98x0.95mm_HandSolder -> NetTie:NetTie-2_SMD_Pad0.5mm
- R2: renamed from R5; value 3.3k -> 3K3
- U2: value HT7533-1 -> HT7333-A; footprint Package_TO_SOT_SMD:SOT-89-3_Handsoldering -> Package_TO_SOT_SMD:SOT-89-3
- Y1: renamed from Y2; value 25 MHz -> CSTNE24M0; footprint Crystal:Crystal_SMD_3225-4Pin_3.2x2.5mm_HandSoldering -> Crystal:Resonator_SMD_Murata_CSTxExxV-3Pin_3.0x1.1mm
- Y2: renamed from Y1; value 32768 12pF -> 32768
- moved J5 11.8 mm to (103.2, 96.0)
- moved R4 6.61 mm to (107.0, 108.3)
- moved J10 6.46 mm to (110.9, 98.0)
- moved C2 5.75 mm to (124.7, 119.7)
- moved C3 5.75 mm to (124.7, 121.2)
- moved J18 3.67 mm to (131.2, 120.2), turned to -90 degrees
- moved NT1 2.44 mm to (132.4, 117.7)
- moved Y1 1.34 mm to (122.0, 104.1), turned to -90 degrees
- moved J4 0.55 mm to (174.9, 103.0)
- moved L1 0.30 mm to (124.7, 118.2)
- moved C7 0.21 mm to (125.6, 101.4)
- renumbered C3 to C1, C21 to C10, C12 to C11, C17 to C12, C18 to C15, C15 to C16, C16 to C17, C4 to C2, C5 to C3, C6 to C4, C7 to C5, C8 to C6, C9 to C7, C10 to C8, C11 to C9, J10 to J11, J11 to J12, J14 to J15, J16 to J17, J7 to J4, J5 to J6, J6 to J7, R2 to R3, R6 to R4
Connections:
- net +3V3 renamed +3.3V
- J12 pad 8: Net-(J11-Pad8) -> unconnected-(J12-Pad8)
- J13 pad 10: Net-(J12-Pad10) -> unconnected-(J13-Pad10)
- J13 pad 6: Net-(J12-Pad6) -> unconnected-(J13-Pad6)
- J3 pad 3: Net-(J3-Pad3) -> unconnected-(J3-Pad3)
- J3 pad 4: Net-(J3-Pad4) -> unconnected-(J3-Pad4)
- J4 pad 2: Net-(J7-Pad2) -> unconnected-(J4-Pad2)
- J4 pad 3: Net-(J7-Pad3) -> unconnected-(J4-Pad3)
- J4 pad 4: Net-(J7-Pad4) -> unconnected-(J4-Pad4)
- J5 pad 1: /TCK -> /JTCK
- J5 pad 4: /TDO -> /JTDO
- J5 pad 6: /RESET -> /JRST
- J9 pad 1: Net-(J9-Pad1) -> unconnected-(J9-Pad1)
- J9 pad 2: Net-(J9-Pad2) -> unconnected-(J9-Pad2)
- SW2 pad 1: Net-(SW2-Pad1) -> unconnected-(SW2-Pad1)
- SW2 pad 4: Net-(SW2-Pad4) -> unconnected-(SW2-Pad4)
Routing:
- net +3.3V: track 231.0 -> 202.6 mm
- net /JTCK: track 20.4 -> 44.9 mm
- net /TDO: track 43.0 -> 27.3 mm
- net /JTDO: track 23.3 -> 37.4 mm
- net /RESET: track 41.0 -> 30.3 mm
- net +3.3VA: track 20.3 -> 29.2 mm
- net /JRXD: track 103.5 -> 94.6 mm, vias 2 -> 1
- net /P5.2: track 15.2 -> 9.19 mm
- net /JTEST: track 48.4 -> 53.8 mm, vias 1 -> 0
- net GNDA: track 17.4 -> 22.2 mm
- net /JTDI: track 50.2 -> 55.0 mm
- net GND: track 53.1 -> 57.8 mm, vias 23 -> 22
- net /JRST: track 18.6 -> 23.3 mm
- net /TCK: track 33.7 -> 30.6 mm
- net /P7.0: track 11.4 -> 8.99 mm
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Other:
- board text added: "RST"
- board text removed: "RESET"

Commit message: Added proto-board production files.
Changed lines of the file:
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@@
       (psa4output false)
       (plotreference true)
-      (plotvalue true)
+      (plotvalue false)
       (plotinvisibletext false)
       (sketchpadsonfab false)
@@
     (fp_line (start 4.52 19.15) (end -1.98 19.15) (layer "F.Fab") (width 0.1))
     (fp_line (start -1.98 5.57) (end -1.98 -3.91) (layer "F.Fab") (width 0.1))
-    (pad "1" thru_hole roundrect locked (at 0 0) (size 1.7 1.7) (drill 1) (layers *.Cu *.Mask) (roundrect_rratio 0.147059)
+    (pad "1" thru_hole roundrect locked (at 0 0) (size 1.7 1.7) (drill 1) (layers *.Cu *.Mask) (roundrect_rratio 0.1470588235)
       (net 55 "/JTDO") (pinfunction "Pin_1") (pintype "passive"))
     (pad "2" thru_hole circle locked (at 2.54 0) (size 1.7 1.7) (drill 1) (layers *.Cu *.Mask)
