File: Hardware/Target_Proto_Boards/SLAU335/SLAU335.kicad_pcb (KiCad board)
At the start: 2 copper layers, 70 x 40 mm, 37 parts, among them J1 USB_B_Micro, J10 GND, J11 +5V, J12 GND, J13 VSEL, J2 LogicAna, J3 DEBUG, J4 PORT1, J5 LED_P2.2, J6 PORT2, J7 JTAG/SBW, J8 AIN, J9 VCC, SW1 TL-2203, SW2 RESET, U1 MSP430I2041TPW, U2 AMS1117-3.3

Commit message: Added proto-board production files.
Other:
- rule pad_to_mask_clearance: 0.1 -> 0
Changed lines of the file:
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@@
   )
   (setup
-    (pad_to_mask_clearance 0.1)
-    (solder_mask_min_width 0.2)
+    (stackup
+      (layer "F.SilkS" (type "Top Silk Screen"))
+      (layer "F.Paste" (type "Top Solder Paste"))
+      (layer "F.Mask" (type "Top Solder Mask") (thickness 0.01))
+      (layer "F.Cu" (type "copper") (thickness 0.035))
+      (layer "dielectric 1" (type "core") (thickness 1.51) (material "FR4") (epsilon_r 4.5) (loss_tangent 0.02))
+      (layer "B.Cu" (type "copper") (thickness 0.035))
+      (layer "B.Mask" (type "Bottom Solder Mask") (thickness 0.01))
+      (copper_finish "None")
+      (dielectric_constraints no)
+    )
+    (pad_to_mask_clearance 0)
     (aux_axis_origin 108 83)
     (grid_origin 108 83)
@@
       (psa4output false)
       (plotreference true)
-      (plotvalue true)
+      (plotvalue false)
       (plotinvisibletext false)
       (sketchpadsonfab false)

Commit message: Fixed regulator part#
Parts:
- U2: value AMS1117-3.3 -> HT7833
