File: Hardware/Target_Proto_Boards/SLAU445_FR2476/FR2476.kicad_pcb (KiCad board)
At the start: 2 copper layers, 70 x 40 mm, 44 parts, among them J1 USB_B_Micro, J10 PORT6, J11 PORT3, J12 JTAG/SBW, J13 VSEL, J14 VCC, J15 GND, J16 +5V, J17 GND, J4 LED_P4.1, J5 DEBUG, J6 PORT4, J7 PORT1, J8 PORT5, J9 PORT2, SW1 TL-2203, SW2 RESET, U1 MSP430FR2476TPTR, U2 AMS1117-3.3, Y1 32768 12pF

Commit message: Added proto-board production files.
Other:
- rule pad_to_mask_clearance: 0.1 -> 0
Changed lines of the file:
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@@
   )
   (setup
-    (pad_to_mask_clearance 0.1)
-    (solder_mask_min_width 0.2)
+    (stackup
+      (layer "F.SilkS" (type "Top Silk Screen"))
+      (layer "F.Paste" (type "Top Solder Paste"))
+      (layer "F.Mask" (type "Top Solder Mask") (thickness 0.01))
+      (layer "F.Cu" (type "copper") (thickness 0.035))
+      (layer "dielectric 1" (type "core") (thickness 1.51) (material "FR4") (epsilon_r 4.5) (loss_tangent 0.02))
+      (layer "B.Cu" (type "copper") (thickness 0.035))
+      (layer "B.Mask" (type "Bottom Solder Mask") (thickness 0.01))
+      (copper_finish "None")
+      (dielectric_constraints no)
+    )
+    (pad_to_mask_clearance 0)
     (grid_origin 108 83)
     (pcbplotparams
@@
       (psa4output false)
       (plotreference true)
-      (plotvalue true)
+      (plotvalue false)
       (plotinvisibletext false)
       (sketchpadsonfab false)

Commit message: Fixed regulator part#
Parts:
- U2: value AMS1117-3.3 -> HT7833
