File: Hardware/STLink-Adapter/STLink-Adapter.kicad_sch (KiCad schematic)
At the start: 7 parts, among them J1 STLINK, J2 SpiBiWire, J3 MSP430, SW1 VCC

Commit message: Final review of 'STLinkV2 Adapter' and fabrication output.
Other:
- company: (none) -> Mathias Gruber
- title: (none) -> STLinkV2 to MSP430 Adapter
Changed lines of the file:
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@@
 (kicad_sch (version 20211123) (generator eeschema)
   (paper "A4")
+  (title_block
+    (title "STLinkV2 to MSP430 Adapter")
+    (date "2022-12-08")
+    (rev "1")
+    (company "Mathias Gruber")
+  )
   (junction (at 83.82 88.9) (diameter 0) (color 0 0 0 0)
   )
