File: Hardware/BluePill-G431/BluePill-G431.kicad_pcb (KiCad board)
At the start: 2 copper layers, 72.5 x 59.7 mm, 41 parts, among them J1 JTAG, J10 Conn_01x12_Male, J2 VCC, J3 GND, J4 SWO, J5 GDB_COMM, J6 TVCC, J7 LogicAna, J8 Conn_01x06_Male, J9 Conn_01x05_Male, U1 BlueAndBlackPill, U2 AD8531ARTZ, U3 74LVC2T45DC, U4 74LS125, U5 74LS125, U6 SRV05-4, U7 SRV05-4

Commit message: New Schematics
Parts:
- added R6: 47K, Resistor_SMD:R_0603_1608Metric_Pad0.98x0.95mm_HandSolder, F.Cu at (153.7, 75.0)
- D1: value LED -> AAA3528SURKCGKS; footprint LED_THT:LED_D3.0mm -> LED_SMD:LED_Kingbright_AAA3528ESGCT
- F1: value 0603L010YR -> 0603L020YR
- J8: value Conn_01x06_Male -> Conn_01x07_Pin; footprint Connector_PinHeader_2.54mm:PinHeader_1x06_P2.54mm_Vertical -> Connector_PinHeader_2.54mm:PinHeader_1x07_P2.54mm_Vertical
- J9: value Conn_01x05_Male -> Conn_01x06_Pin; footprint Connector_PinHeader_2.54mm:PinHeader_1x05_P2.54mm_Vertical -> Connector_PinHeader_2.54mm:PinHeader_1x06_P2.54mm_Vertical
- R5: value 1K -> 180
- U1: value BlueAndBlackPill -> BluePillAndG431; footprint lib:BlueBlackPill -> lib:BluePillG431
- moved J3 2.62 mm to (160.0, 70.0)
- moved J6 2.51 mm to (185.4, 70.1)
- moved J2 2.50 mm to (171.4, 70.1)
- moved J9 2.50 mm to (123.2, 93.0)
- moved R5 1.42 mm to (123.5, 114.9), turned to -90 degrees
- moved D1 1.15 mm to (122.0, 110.8), turned to 0 degrees
- moved U1 0.07 mm to (129.6, 70.0)
- renumbered C3 to C1, C11 to C10, C10 to C11, C1 to C2, C5 to C3, C2 to C4, C4 to C5, C7 to C6, C6 to C7
Connections:
- net /JRST renamed /t.RST
- net /JRXD renamed /t.RXD
- net /JTCK renamed /t.TCK
- net /JTDI renamed /t.TDI
- net /JTDO renamed /t.TDO
- net /JTEST renamed /t.TEST
- net /JTMS renamed /t.TMS
- net /JTXD renamed /t.TXD
- net /rRST renamed /r.RST
- net /rRXD renamed /r.RXD
- net /rTCK renamed /r.TCK
- net /rTDI renamed /r.TDI
- net /rTDO renamed /r.TDO
- net /rTEST renamed /r.TEST
- net /rTMS renamed /r.TMS
- net /rTXD renamed /r.TXD
- C5 pad 2: /VREF_2 -> /V2REF
- C7 pad 2: VCC -> Net-(U2--)
- D1 pad 2: Net-(D1-Pad2) -> Net-(D1-A1)
- F1 pad 1: Net-(F1-Pad1) -> Net-(U2--)
- J10 pad 1: /PB10 -> /DIS_TCK
- J10 pad 10: /mRST -> /h.RST
- J10 pad 11: /VREF_2 -> /V2REF
- J10 pad 12: /LEDS -> GND
- J10 pad 2: /PB1 -> /DIS_RST
- J10 pad 3: /PB0 -> /PB1
- J10 pad 4: /mTDI -> /h.TDI
- J10 pad 5: /mTDO -> /h.TDO
- J10 pad 6: /mTCK -> /h.TCK
- J10 pad 7: /mTEST -> /h.TEST
- J10 pad 8: /mRXD -> /h.TXD
- J10 pad 9: /mTXD -> /h.RXD
- J7 pad 1: /mTMS -> /h.TMS
- J7 pad 2: /mTCK -> /h.TCK
- J7 pad 3: /mTDI -> /h.TDI
- J7 pad 4: /mTDO -> /h.TDO
- J7 pad 5: /mTEST -> /h.TEST
- J7 pad 6: /mRST -> /h.RST
- J8 pad 1: /ENA1N -> /DIS_JTAG
- J8 pad 2: /ENA2N -> /DIS_COM
- J8 pad 3: /ENA3N -> /PB14
- J8 pad 5: /mTCK -> /h.TCK
- J8 pad 6: /SBWO -> /h.TMS
- J9 pad 1: /mTMS -> /SBW_RD
- J9 pad 4: /TV_PWM -> /PB8
- J9 pad 5: /PB9 -> /GEN_VT
- R1 pad 2: /TV_PWM -> /GEN_VT
- R2 pad 2: /TV_PWM -> /GEN_VT
- R3 pad 1: /VREF_2 -> /V2REF
- R4 pad 2: /VREF_2 -> /V2REF
- R5 pad 1: Net-(D1-Pad2) -> Net-(D1-A1)
- RN1 pad 1: /ENA1N -> /DIS_RST
- RN1 pad 2: /ENA2N -> /DIS_JTAG
- RN1 pad 3: /ENA3N -> /DIS_COM
- RN1 pad 4: /SBWO -> /SBW_RD
- RN1 pad 5: GND -> +3V3
- RN1 pad 6: GND -> +3V3
- RN1 pad 7: GND -> +3V3
- RN1 pad 8: GND -> +3V3
- U1 pad A1: /ENA1N -> /DIS_JTAG
- U1 pad A10: unconnected-(U1-PadA10) -> /LEDS
- U1 pad A14: /GDB_TX -> /h.TXD
- U1 pad A15: /GDB_RX -> /h.RXD
- U1 pad A16: /TV_PWM -> /PB8
- U1 pad A17: /PB9 -> /GEN_VT
- U1 pad A2: /ENA2N -> /DIS_COM
- U1 pad A22: /LEDS -> unconnected-(U1A-PC13-PadA22)
- U1 pad A25: /VREF_2 -> /h.TEST
- U1 pad A26: /mRST -> /h.RST
- U1 pad A27: /mTXD -> /GDB_TX
- U1 pad A28: /mRXD -> /GDB_RX
- U1 pad A29: /mTEST -> /GEN_VT
- U1 pad A3: /ENA3N -> /PB14
- U1 pad A30: /mTCK -> /h.TCK
- U1 pad A31: /mTDO -> /h.TDO
- U1 pad A32: /mTDI -> /h.TDI
- U1 pad A33: /PB0 -> /V2REF
- U1 pad A35: /PB10 -> /DIS_RST
- U1 pad A36: unconnected-(U1-PadA36) -> /DIS_TCK
- U1 pad A5: /mTCK -> /h.TCK
- U1 pad A6: /SBWO -> /h.TMS
- U1 pad A7: /mTMS -> /SBW_RD
- U1 pad B1: /ENA1N -> /DIS_JTAG
- U1 pad B10: unconnected-(U1-PadB10) -> /LEDS
- U1 pad B14: /GDB_TX -> /h.TXD
- U1 pad B15: /GDB_RX -> /h.RXD
- U1 pad B16: /TV_PWM -> /PB8
- U1 pad B17: /PB9 -> /GEN_VT
- U1 pad B2: /ENA2N -> /DIS_COM
- U1 pad B22: /LEDS -> unconnected-(U1B-PC13-PadB22)
- U1 pad B25: unconnected-(U1-PadB25) -> /h.TEST
- U1 pad B26: /VREF_2 -> /h.RST
- U1 pad B27: /mRST -> /GDB_TX
- U1 pad B28: /mTXD -> /GDB_RX
- U1 pad B29: /mRXD -> /GEN_VT
- U1 pad B3: /ENA3N -> /PB14
- U1 pad B30: /mTEST -> /h.TCK
- U1 pad B31: /mTCK -> /h.TDO
- U1 pad B32: /mTDO -> /h.TDI
- U1 pad B33: /mTDI -> /V2REF
- U1 pad B34: /PB0 -> /PB1
- U1 pad B35: /PB1 -> unconnected-(U1B-PB2-PadB35)
- U1 pad B36: unconnected-(U1-PadB36) -> /DIS_RST
- U1 pad B37: /PB10 -> /DIS_TCK
- U1 pad B38: +3V3 -> unconnected-(U1B-NRST-PadB38)
- U1 pad B39: GND -> +3V3
- U1 pad B40: unconnected-(U1-PadB40) -> GND
- U1 pad B5: /mTCK -> /h.TCK
- U1 pad B6: /SBWO -> /h.TMS
- U1 pad B7: /mTMS -> /SBW_RD
- U2 pad 1: Net-(F1-Pad1) -> Net-(U2--)
- U2 pad 4: VCC -> Net-(U2--)
- U3 pad 2: /mTDO -> /h.TDO
- U3 pad 3: /mRXD -> /h.RXD
- U4 pad 10: /SBWO -> /SBW_RD
- U4 pad 12: /mTDI -> /h.TDI
- U4 pad 13: /ENA2N -> /DIS_JTAG
- U4 pad 4: /ENA2N -> /DIS_JTAG
- U4 pad 5: /mTMS -> /h.TMS
- U4 pad 9: /mTDI -> /h.TDI
- U5 pad 1: /ENA1N -> /DIS_RST
- U5 pad 10: /ENA1N -> /DIS_TCK
- U5 pad 12: /mRST -> /h.RST
- U5 pad 13: /ENA1N -> /DIS_RST
- U5 pad 2: /mTEST -> /h.TEST
- U5 pad 4: /ENA3N -> /DIS_COM
- U5 pad 5: /mTXD -> /h.TXD
- U5 pad 9: /mTCK -> /h.TCK
Routing:
- net /h.TCK: track 0.00 -> 86.2 mm, vias 0 -> 1
- net /SBW_RD: track 0.00 -> 82.9 mm, vias 0 -> 3
- net /mTCK: track 81.0 -> 0.00 mm
- net /ENA1N: track 80.4 -> 0.00 mm, vias 3 -> 0
- net /GEN_VT: track 0.00 -> 76.7 mm, vias 0 -> 2
- net /ENA3N: track 75.4 -> 0.00 mm, vias 2 -> 0
- net /mTMS: track 72.9 -> 0.00 mm
- net /h.TMS: track 0.00 -> 71.6 mm, vias 0 -> 1
- net /DIS_COM: track 0.00 -> 70.4 mm, vias 0 -> 2
- net /SBWO: track 69.9 -> 0.00 mm, vias 2 -> 0
- net /ENA2N: track 63.7 -> 0.00 mm, vias 3 -> 0
- net /DIS_JTAG: track 0.00 -> 62.5 mm, vias 0 -> 3
- net /TV_PWM: track 62.4 -> 0.00 mm
- net /h.TEST: track 0.00 -> 62.0 mm, vias 0 -> 1
- net /h.TXD: track 0.00 -> 59.1 mm
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Other:
- board text added: "BlueBill+G431 Glossy-MSP430"
- board text added: "G1"
- board text added: "G431"
- board text added: "GEN.V"
- board text added: "PB14"
- board text added: "PB8"
- board text added: "SBW.R"
- board text added: "~{dCOM}"
- board text added: "~{dJTAG}"
- board text added: "~{dRST}"
- board text added: "~{dTCK}"
- board text added: "©2026 by GruMat github.com/grumat/glossy-msp430.git"
- board text removed: "BlackPill"
- board text removed: "Blue+BlackBill Glossy-MSP430"
- board text removed: "LEDS"
- board text removed: "PB0"
- board text removed: "PB10"
- board text removed: "PB9"
- board text removed: "TVpwm"
- board text removed: "V2"
- board text removed: "~{ENA1}"
- board text removed: "~{ENA2}"
- board text removed: "~{ENA3}"
- board text removed: "~{SBWO}"
- board text removed: "©2022 by GruMat github.com/grumat/glossy-msp430.git"

Commit message: Added fabrication files
Parts:
- moved D1 8.90 mm to (121.9, 119.7)
- moved R5 0.34 mm to (123.5, 115.2), turned to 90 degrees
Routing:
- net GND: track 150.5 -> 166.4 mm, vias 41 -> 43
- net +3V3: track 211.1 -> 215.0 mm
- net /LEDS: track 30.0 -> 29.4 mm

Commit message: Version 1.1 of Bluepill/G431
Parts:
- D1: footprint LED_SMD:LED_Kingbright_AAA3528ESGCT -> LED_SMD:LED_Avago_PLCC4_3.2x2.8mm_CW
- R5: value 180 -> 150
- R6: value 47K -> 10K
- RN1, RN2, RN4: value 47k -> 10k; footprint Resistor_SMD:R_Array_Convex_4x0402 -> lib:EXB38V_PAN-M
- RN3, RN5: value 100 -> 33; footprint Resistor_SMD:R_Array_Convex_4x0402 -> lib:EXB38V_PAN-M
- moved U6 7.54 mm to (178.1, 78.0)
- moved RN3 5.60 mm to (178.5, 83.7)
- moved RN5 3.18 mm to (178.5, 95.4)
- moved RN2 3.06 mm to (178.5, 89.5)
- moved J1 2.54 mm to (185.4, 87.9)
- moved RN4 1.46 mm to (178.5, 101.2)
- moved RN1 0.81 mm to (163.0, 77.2)
Routing:
- net VCC: track 142.4 -> 151.6 mm, vias 9 -> 8
- net /r.TDI: track 23.9 -> 31.2 mm, vias 2 -> 3
- net /r.TMS: track 17.8 -> 25.0 mm
- net /r.RST: track 13.2 -> 18.9 mm, vias 0 -> 2
- net /t.RXD: track 10.5 -> 15.9 mm
- net /t.RST: track 24.0 -> 28.8 mm
- net /t.TDI: track 5.98 -> 10.8 mm
- net /r.TEST: track 23.1 -> 27.9 mm
- net /r.TXD: track 17.8 -> 22.5 mm
- net /t.TMS: track 7.88 -> 12.5 mm
- net /r.TCK: track 24.2 -> 28.0 mm
- net /t.TDO: track 5.57 -> 9.23 mm
- net GND: track 166.4 -> 162.9 mm, vias 43 -> 44
- net /t.TXD: track 8.73 -> 11.3 mm
- net /r.RXD: track 12.9 -> 14.7 mm
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Other:
- board size 72.5 x 59.7 mm -> 74.9 x 59.7 mm
